Commit message: penambahan teleop, robot sekarang dapat di kontrol di terminal melalui keyboard

File: src/my_robot/description/urdf/robot.xacro (robot description, xacro)
@@ -100,16 +100,18 @@
       </geometry>
     </visual>
-  	<collision name="caster_cylinder">
-    	<origin xyz="0 0 -0.002" rpy="0 0 0"/>
-    	<geometry>
-    	  <cylinder radius="0.007850" length="0.012"/>
-    	</geometry>
-  	</collision>
-  	<collision name="caster_sphere">
-    	<origin xyz="0 0 -0.009" rpy="0 0 0"/>
-    	<geometry>
-      	  <sphere radius="0.006"/>
-    	</geometry>
-  	</collision>
+    <collision>
+      <origin xyz="0 0 -0.008" rpy="0 0 0"/>
+      <geometry>
+        <sphere radius="0.006"/>
+      </geometry>
+      <surface>
+        <friction>
+          <ode>
+            <mu>0.05</mu>
+            <mu2>0.05</mu2>
+          </ode>
+        </friction>
+      </surface>
+    </collision>
   </link>
   <joint name="caster_joint" type="fixed">

Commit message: Checkpoint 1, pergerakan robot sudah cukup baik walau terkadang terdapat beberapa bug, dan beberapa fitur sudah dapat digunakan (cek README.md)

File: src/my_robot/description/urdf/robot.xacro (robot description, xacro)
@@ -14,7 +14,7 @@
   <xacro:property name="y_imu" value="0.0"/>
   <xacro:property name="z_imu" value="0.024"/>
-  <xacro:property name="mu_drive" value="1.6"/>
+  <xacro:property name="mu_drive" value="0.8"/>
   <xacro:property name="mu_caster" value="0.0"/>
-  <xacro:property name="wheel_damping" value="0.1"/>
+  <xacro:property name="wheel_damping" value="0.5"/>
   <xacro:property name="wheel_left_slip1" value="0.00"/>
   <xacro:property name="wheel_left_slip2" value="0.00"/>
@@ -221,4 +221,8 @@
       <wheel_separation>0.104</wheel_separation>
       <wheel_radius>0.02131869</wheel_radius>
+      <max_linear_velocity>1.0</max_linear_velocity>
+      <max_angular_velocity>2.0</max_angular_velocity>
+      <linear_acceleration_limit>1.0</linear_acceleration_limit>
+      <angular_acceleration_limit>2.0</angular_acceleration_limit>
       <topic>/cmd_vel</topic>
       <odom_topic>/odom</odom_topic>
@@ -226,4 +230,6 @@
       <frame_id>odom</frame_id>
       <child_frame_id>base_link</child_frame_id>
+      <publish_wheel_tf>false</publish_wheel_tf>
+      <publish_odom_tf>true</publish_odom_tf>
     </plugin>
   </gazebo>

Commit message: backup terakhir sebelum mencoba menghapus semua design dan menggunakan design sederhana

File: src/my_robot/description/urdf/robot.xacro (robot description, xacro)
@@ -14,16 +14,19 @@
   <xacro:property name="y_imu" value="0.0"/>
   <xacro:property name="z_imu" value="0.024"/>
-  <xacro:property name="mu_drive" value="0.8"/>
-  <xacro:property name="mu_caster" value="0.0"/>
-  <xacro:property name="wheel_damping" value="0.5"/>
-  <xacro:property name="wheel_left_slip1" value="0.00"/>
-  <xacro:property name="wheel_left_slip2" value="0.00"/>
-  <xacro:property name="wheel_right_slip1" value="0.00"/>
-  <xacro:property name="wheel_right_slip2" value="0.00"/>
+  <!-- UPDATED PARAMETERS -->
+  <xacro:property name="mu_drive" value="1.0"/>
+  <xacro:property name="mu_drive_lateral" value="1.3"/>
+  <xacro:property name="mu_caster" value="0.1"/>
+  <xacro:property name="wheel_damping" value="1.5"/>
+  <xacro:property name="wheel_left_slip1" value="0.005"/>
+  <xacro:property name="wheel_left_slip2" value="0.005"/>
+  <xacro:property name="wheel_right_slip1" value="0.005"/>
+  <xacro:property name="wheel_right_slip2" value="0.005"/>
   <!-- ================= BASE ================= -->
   <link name="base_link">
     <inertial>
       <mass value="2.0"/>
-      <origin xyz="0 0 0" rpy="0 0 0"/>
+      <!-- LOWERED CoM -->
+      <origin xyz="0 0 -0.01" rpy="0 0 0"/>
       <inertia ixx="0.01" iyy="0.015" izz="0.02"
                ixy="0" ixz="0" iyz="0"/>
@@ -47,5 +50,6 @@
       <mass value="0.2"/>
       <origin xyz="0 0 0" rpy="0 0 0"/>
-      <inertia ixx="0.0001" iyy="0.0001" izz="0.0001"
+      <!-- IMPROVED INERTIA -->
+      <inertia ixx="0.0002" iyy="0.0001" izz="0.0002"
                ixy="0" ixz="0" iyz="0"/>
     </inertial>
@@ -65,7 +69,8 @@
           <ode>
             <mu>${mu_drive}</mu>
-            <mu2>${mu_drive}</mu2>
+            <mu2>${mu_drive_lateral}</mu2>
             <slip1>${wheel_left_slip1}</slip1>
             <slip2>${wheel_left_slip2}</slip2>
+            <fdir1>1 0 0</fdir1>
           </ode>
         </friction>
@@ -85,5 +90,6 @@
       <mass value="0.2"/>
       <origin xyz="0 0 0" rpy="0 0 0"/>
-      <inertia ixx="0.0001" iyy="0.0001" izz="0.0001"
+      <!-- IMPROVED INERTIA -->
+      <inertia ixx="0.0002" iyy="0.0001" izz="0.0002"
                ixy="0" ixz="0" iyz="0"/>
     </inertial>
@@ -103,7 +109,8 @@
           <ode>
             <mu>${mu_drive}</mu>
-            <mu2>${mu_drive}</mu2>
+            <mu2>${mu_drive_lateral}</mu2>
             <slip1>${wheel_right_slip1}</slip1>
             <slip2>${wheel_right_slip2}</slip2>
+            <fdir1>1 0 0</fdir1>
           </ode>
         </friction>
