Commit message: penambahan imu dan selesai perbaikan design .xacro robot untuk sesuai dengan kinematika

File: src/my_robot/description/urdf/robot.urdf (robot description, URDF)
Before this commit: robot my_robot, 4 links, 3 joints
Links:
- added link imu_link, mass 0.01
- link base_link: geometry collision box size=0.099 0.086 0.05379345; visual mesh filename=package://my_robot/description/meshes/body.dae scale=1.0 1.0 1.0
- link caster_wheel: geometry collision sphere radius=0.006; visual mesh filename=package://my_robot/description/meshes/freewheel.dae scale=1.0 1.0 1.0
Joints:
- added joint imu_joint: type fixed, parent base_link, child imu_link, origin xyz=0.0 0.0 0.02 rpy=0 0 0
- joint caster_joint: origin xyz=0.0 -0.038 0.0 rpy=0 0 0 -> xyz=0.038 0.0 0.0 rpy=0 0 0
- joint left_wheel_joint: axis 1 0 0 -> 0 1 0; origin xyz=0.052 0.029 0.008 rpy=0 0 0 -> xyz=-0.029 0.052 0.008 rpy=0 0 0
- joint right_wheel_joint: axis 1 0 0 -> 0 1 0; origin xyz=-0.052 0.029 0.008 rpy=0 0 0 -> xyz=-0.029 -0.052 0.008 rpy=0 0 0

File: src/my_robot/description/urdf/robot.xacro (robot description, xacro)
@@ -2,13 +2,23 @@
 <robot name="my_robot" xmlns:xacro="http://www.ros.org/wiki/xacro">
   <!-- ================= PROPERTIES ================= -->
-  <xacro:property name="x_l" value="0.052"/>
-  <xacro:property name="y_l" value="0.029"/>
+  <xacro:property name="x_l" value="-0.029"/>
+  <xacro:property name="y_l" value="0.052"/>
   <xacro:property name="z_l" value="0.008"/>
-  <xacro:property name="x_r" value="-0.052"/>
-  <xacro:property name="y_r" value="0.029"/>
+  <xacro:property name="x_r" value="-0.029"/>
+  <xacro:property name="y_r" value="-0.052"/>
   <xacro:property name="z_r" value="0.008"/>
-  <xacro:property name="x_c" value="0.00"/>
-  <xacro:property name="y_c" value="-0.038"/>
+  <xacro:property name="x_c" value="0.038"/>
+  <xacro:property name="y_c" value="0.00"/>
   <xacro:property name="z_c" value="0.00"/>
+  <xacro:property name="x_imu" value="0.0"/>
+  <xacro:property name="y_imu" value="0.0"/>
+  <xacro:property name="z_imu" value="0.02"/>
+  <xacro:property name="mu_drive" value="1.6"/>
+  <xacro:property name="mu_caster" value="0.0"/>
+  <xacro:property name="wheel_damping" value="0.1"/>
+  <xacro:property name="wheel_left_slip1" value="0.00"/>
+  <xacro:property name="wheel_left_slip2" value="0.00"/>
+  <xacro:property name="wheel_right_slip1" value="0.00"/>
+  <xacro:property name="wheel_right_slip2" value="0.00"/>
   <!-- ================= BASE ================= -->
   <link name="base_link">
@@ -20,5 +30,5 @@
     </inertial>
     <visual>
-      <origin xyz="0 0 0" rpy="0 0 0"/>
+      <origin xyz="0 0 0" rpy="0 0 1.5708"/>
       <geometry>
         <mesh filename="package://my_robot/description/meshes/body.dae" scale="1.0 1.0 1.0"/>
@@ -28,5 +38,5 @@
       <origin xyz="0 0 0.026" rpy="0 0 0"/>
       <geometry>
-        <box size="0.086 0.099 0.05379345"/>
+        <box size="0.099 0.086 0.05379345"/>
       </geometry>
     </collision>
@@ -41,5 +51,5 @@
     </inertial>
     <visual>
-      <origin xyz="0 0 0" rpy="0 0 0"/>
+      <origin xyz="0 0 0" rpy="0 0 1.5708"/>
       <geometry>
         <mesh filename="package://my_robot/description/meshes/roda2.dae" scale="1.0 1.0 1.0"/>
@@ -47,67 +57,15 @@
     </visual>
     <collision>
-      <origin xyz="0 0 0" rpy="0 1.5708 0"/>
+      <origin xyz="0 0 0" rpy="1.5708 0 0"/>
       <geometry>
         <cylinder radius="0.02131869" length="0.017"/>
-      </geometry>
-    </collision>
-  </link>
-  <joint name="left_wheel_joint" type="continuous">
-    <parent link="base_link"/>
-    <child link="left_wheel"/>
-    <origin xyz="${x_l} ${y_l} ${z_l}" rpy="0 0 0"/>
-    <axis xyz="1 0 0"/>
-  </joint>
-  <!-- ================= RIGHT WHEEL ================= -->
-  <link name="right_wheel">
-    <inertial>
-      <mass value="0.2"/>
-      <origin xyz="0 0 0" rpy="0 0 0"/>
-      <inertia ixx="0.0001" iyy="0.0001" izz="0.0001"
-               ixy="0" ixz="0" iyz="0"/>
-    </inertial>
-    <visual>
-      <origin xyz="0 0 0" rpy="0 0 0"/>
-      <geometry>
-        <mesh filename="package://my_robot/description/meshes/roda1.dae" scale="1.0 1.0 1.0"/>
-      </geometry>
-    </visual>
-    <collision>
-      <origin xyz="0 0 0" rpy="0 1.5708 0"/>
-      <geometry>
-        <cylinder radius="0.02131869" length="0.017"/>
-      </geometry>
-    </collision>
-  </link>
-  <joint name="right_wheel_joint" type="continuous">
-    <parent link="base_link"/>
-    <child link="right_wheel"/>
-    <origin xyz="${x_r} ${y_r} ${z_r}" rpy="0 0 0"/>
-    <axis xyz="1 0 0"/>
-  </joint>
-  <!-- ================= CASTER ================= -->
-  <link name="caster_wheel">
-    <inertial>
-      <mass value="0.1"/>
-      <origin xyz="0 0 0" rpy="0 0 0"/>
-      <inertia ixx="0.00001" iyy="0.00001" izz="0.00001"
-               ixy="0" ixz="0" iyz="0"/>
-    </inertial>
-    <visual>
-      <origin xyz="0 0 0" rpy="0 0 0"/>
-      <geometry>
-        <mesh filename="package://my_robot/description/meshes/freewheel.dae" scale="1.0 1.0 1.0"/>
-      </geometry>
-    </visual>
-    <collision>
-      <origin xyz="0 0 -0.008" rpy="0 0 0"/>
-      <geometry>
-        <sphere radius="0.006"/>
       </geometry>
       <surface>
         <friction>
           <ode>
-            <mu>0.05</mu>
-            <mu2>0.05</mu2>
+            <mu>${mu_drive}</mu>
+            <mu2>${mu_drive}</mu2>
+            <slip1>${wheel_left_slip1}</slip1>
+            <slip2>${wheel_left_slip2}</slip2>
           </ode>
         </friction>
@@ -115,4 +73,78 @@
     </collision>
   </link>
+  <joint name="left_wheel_joint" type="continuous">
+    <parent link="base_link"/>
+    <child link="left_wheel"/>
+    <origin xyz="${x_l} ${y_l} ${z_l}" rpy="0 0 0"/>
+    <axis xyz="0 1 0"/>
+    <dynamics damping="${wheel_damping}" friction="0.0"/>
+  </joint>
+  <!-- ================= RIGHT WHEEL ================= -->
+  <link name="right_wheel">
+    <inertial>
+      <mass value="0.2"/>
+      <origin xyz="0 0 0" rpy="0 0 0"/>
+      <inertia ixx="0.0001" iyy="0.0001" izz="0.0001"
+               ixy="0" ixz="0" iyz="0"/>
+    </inertial>
+    <visual>
+      <origin xyz="0 0 0" rpy="0 0 1.5708"/>
+      <geometry>
+        <mesh filename="package://my_robot/description/meshes/roda1.dae" scale="1.0 1.0 1.0"/>
+      </geometry>
+    </visual>
+    <collision>
+      <origin xyz="0 0 0" rpy="1.5708 0 0"/>
+      <geometry>
+        <cylinder radius="0.02131869" length="0.017"/>
+      </geometry>
+      <surface>
+        <friction>
+          <ode>
+            <mu>${mu_drive}</mu>
+            <mu2>${mu_drive}</mu2>
+            <slip1>${wheel_right_slip1}</slip1>
+            <slip2>${wheel_right_slip2}</slip2>
+          </ode>
+        </friction>
+      </surface>
+    </collision>
+  </link>
+  <joint name="right_wheel_joint" type="continuous">
+    <parent link="base_link"/>
+    <child link="right_wheel"/>
+    <origin xyz="${x_r} ${y_r} ${z_r}" rpy="0 0 0"/>
+    <axis xyz="0 1 0"/>
+    <dynamics damping="${wheel_damping}" friction="0.0"/>
+  </joint>
+  <!-- ================= CASTER ================= -->
+  <link name="caster_wheel">
+    <inertial>
+      <mass value="0.1"/>
+      <origin xyz="0 0 0" rpy="0 0 0"/>
+      <inertia ixx="0.00001" iyy="0.00001" izz="0.00001"
+               ixy="0" ixz="0" iyz="0"/>
+    </inertial>
+    <visual>
+      <origin xyz="0 0 0" rpy="0 0 0"/>
+      <geometry>
+        <mesh filename="package://my_robot/description/meshes/freewheel.dae" scale="1.0 1.0 1.0"/>
+      </geometry>
+    </visual>
+    <collision>
+      <origin xyz="0 0 -0.008" rpy="0 0 0"/>
+      <geometry>
+        <sphere radius="0.006"/>
+      </geometry>
+      <surface>
+        <friction>
+          <ode>
+            <mu>${mu_caster}</mu>
+            <mu2>${mu_caster}</mu2>
+          </ode>
+        </friction>
+      </surface>
+    </collision>
+  </link>
   <joint name="caster_joint" type="fixed">
     <parent link="base_link"/>
@@ -120,4 +152,67 @@
     <origin xyz="${x_c} ${y_c} ${z_c}" rpy="0 0 0"/>
   </joint>
+  <!-- ================= IMU ================= -->
+  <link name="imu_link">
+    <inertial>
+      <mass value="0.01"/>
+      <origin xyz="0 0 0" rpy="0 0 0"/>
+      <inertia ixx="0.000001" iyy="0.000001" izz="0.000001"
+               ixy="0" ixz="0" iyz="0"/>
+    </inertial>
+  </link>
+  <joint name="imu_joint" type="fixed">
+    <parent link="base_link"/>
+    <child link="imu_link"/>
+    <origin xyz="${x_imu} ${y_imu} ${z_imu}" rpy="0 0 0"/>
+  </joint>
+  <gazebo reference="imu_link">
+    <sensor name="imu_sensor" type="imu">
+      <always_on>true</always_on>
+      <update_rate>100</update_rate>
+      <topic>/imu</topic>
+      <imu>
+        <angular_velocity>
+          <x>
+            <noise type="gaussian">
+              <mean>0.0</mean>
+              <stddev>0.0002</stddev>
+            </noise>
+          </x>
+          <y>
+            <noise type="gaussian">
+              <mean>0.0</mean>
+              <stddev>0.0002</stddev>
+            </noise>
+          </y>
+          <z>
+            <noise type="gaussian">
+              <mean>0.0</mean>
+              <stddev>0.0002</stddev>
+            </noise>
+          </z>
+        </angular_velocity>
+        <linear_acceleration>
+          <x>
+            <noise type="gaussian">
+              <mean>0.0</mean>
+              <stddev>0.017</stddev>
+            </noise>
+          </x>
+          <y>
+            <noise type="gaussian">
+              <mean>0.0</mean>
+              <stddev>0.017</stddev>
+            </noise>
+          </y>
+          <z>
+            <noise type="gaussian">
+              <mean>0.0</mean>
+              <stddev>0.017</stddev>
+            </noise>
+          </z>
+        </linear_acceleration>
+      </imu>
+    </sensor>
+  </gazebo>
   <gazebo>
     <plugin filename="gz-sim-diff-drive-system" name="gz::sim::systems::DiffDrive">

Commit message: fix sensor imu tidak terdeteksi, sekarang sensor imu sudah bekerja sebagaimana mestinya

File: src/my_robot/description/urdf/robot.urdf (robot description, URDF)
Before this commit: robot my_robot, 5 links, 4 joints
Joints:
- joint imu_joint: origin xyz=0.0 0.0 0.02 rpy=0 0 0 -> xyz=0.033 0.0 0.024 rpy=0 0 0

File: src/my_robot/description/urdf/robot.xacro (robot description, xacro)
@@ -11,7 +11,7 @@
   <xacro:property name="y_c" value="0.00"/>
   <xacro:property name="z_c" value="0.00"/>
-  <xacro:property name="x_imu" value="0.0"/>
+  <xacro:property name="x_imu" value="0.033"/>
   <xacro:property name="y_imu" value="0.0"/>
-  <xacro:property name="z_imu" value="0.02"/>
+  <xacro:property name="z_imu" value="0.024"/>
   <xacro:property name="mu_drive" value="1.6"/>
   <xacro:property name="mu_caster" value="0.0"/>

Commit message: Selesai perbaikan pergerakan robot, sekarang behaviour pergerakan robot sesuai dengan yang diinginkan

File: src/my_robot/description/urdf/robot.urdf (robot description, URDF)
Before this commit: robot my_robot, 5 links, 4 joints
Links:
- link caster_wheel: mass 0.1 -> 0.02

File: src/my_robot/description/urdf/robot.xacro (robot description, xacro)
@@ -17,5 +17,7 @@
   <xacro:property name="mu_drive" value="1.0"/>
   <xacro:property name="mu_drive_lateral" value="1.3"/>
-  <xacro:property name="mu_caster" value="0.1"/>
+  <xacro:property name="mu_caster" value="0.01"/>
+  <xacro:property name="caster_slip1" value="0.15"/>
+  <xacro:property name="caster_slip2" value="0.15"/>
   <xacro:property name="wheel_damping" value="1.5"/>
   <xacro:property name="wheel_left_slip1" value="0.005"/>
@@ -27,6 +29,5 @@
     <inertial>
       <mass value="2.0"/>
-      <!-- LOWERED CoM -->
-      <origin xyz="0 0 -0.01" rpy="0 0 0"/>
+      <origin xyz="-0.015 0 0" rpy="0 0 0"/>
       <inertia ixx="0.01" iyy="0.015" izz="0.02"
                ixy="0" ixz="0" iyz="0"/>
@@ -128,7 +129,7 @@
   <link name="caster_wheel">
     <inertial>
-      <mass value="0.1"/>
-      <origin xyz="0 0 0" rpy="0 0 0"/>
-      <inertia ixx="0.00001" iyy="0.00001" izz="0.00001"
+      <mass value="0.02"/>
+      <origin xyz="0 0 0" rpy="0 0 0"/>
+      <inertia ixx="0.000002" iyy="0.000002" izz="0.000002"
                ixy="0" ixz="0" iyz="0"/>
     </inertial>
@@ -140,5 +141,5 @@
     </visual>
     <collision>
-      <origin xyz="0 0 -0.008" rpy="0 0 0"/>
+      <origin xyz="0 0 -0.007" rpy="0 0 0"/>
       <geometry>
         <sphere radius="0.006"/>
@@ -149,4 +150,6 @@
             <mu>${mu_caster}</mu>
             <mu2>${mu_caster}</mu2>
+            <slip1>${caster_slip1}</slip1>
+            <slip2>${caster_slip2}</slip2>
           </ode>
         </friction>
